Commit message: Update SLAM configuration and improve coverage planner
- Changed SLAM mode from 'mapping' to 'lifelong' in slam_toolbox.yaml for continuous mapping.
- Updated launch files (full_system.launch.py, navigation.launch.py, sim_full_system.launch.py) to set default SLAM mode to 'lifelong' and specify the map file name.
- Enhanced navigation.launch.py to support 'lifelong' mode with appropriate parameter rewrites.
- Modified coverage planner to handle obstacle polygons and ensure headland width meets minimum turning radius requirements.
- Updated map server to manage multiple allowed area polygons and obstacle polygons for better navigation and coverage planning.
- Removed small obstacles from the simulation world (garden.sdf) that are less than 40cm in height to improve robot navigation.

File: src/mowgli_bringup/urdf/mowgli.urdf.xacro (robot description, xacro)
@@ -8,10 +8,10 @@
     y  left
     z  up
-  Key dimensions:
-    Base:          0.55 m long, 0.40 m wide, 0.25 m high
-    Drive wheels:  radius 0.10 m, width 0.05 m, track 0.35 m
-    Caster:        radius 0.04 m (front)
-    Blade disc:    radius 0.15 m, height 0.02 m (centred under base)
-    Wheel ground clearance sets base_link at z = wheel_radius = 0.10 m
+  Key dimensions (from real YardForce Classic 500 URDF):
+    Base:          0.54 m long, 0.40 m wide, 0.19 m high
+    Drive wheels:  radius 0.04475 m, width 0.04 m, track 0.40 m (rear)
+    Front casters: radius 0.03 m, width 0.03 m
+    Blade disc:    radius 0.09 m, height 0.01 m (centred under base)
+    Wheel ground clearance sets base_link at z = drive_wheel_radius = 0.04475 m
     above base_footprint.
 -->
@@ -20,16 +20,23 @@
        Properties
        ================================================================ -->
-  <xacro:property name="base_length"     value="0.55"/>
+  <xacro:property name="base_length"     value="0.54"/>
   <xacro:property name="base_width"      value="0.40"/>
-  <xacro:property name="base_height"     value="0.25"/>
-  <xacro:property name="wheel_radius"    value="0.10"/>
-  <xacro:property name="wheel_width"     value="0.05"/>
-  <xacro:property name="wheel_track"     value="0.35"/>  <!-- centre-to-centre -->
+  <xacro:property name="base_height"     value="0.19"/>
+  <!-- Rear drive wheels (from real URDF: diameter 0.0895m) -->
+  <xacro:property name="wheel_radius"    value="0.04475"/>
+  <xacro:property name="wheel_width"     value="0.04"/>
+  <xacro:property name="wheel_track"     value="0.40"/>  <!-- centre-to-centre -->
   <xacro:property name="wheel_mass"      value="0.5"/>
-  <xacro:property name="caster_radius"   value="0.04"/>
+  <!-- Rear wheels are offset behind base_link centre -->
+  <xacro:property name="wheel_x_offset"  value="-0.18"/>
+  <!-- Front caster wheels (smaller) -->
+  <xacro:property name="caster_radius"   value="0.03"/>
+  <xacro:property name="caster_width"    value="0.03"/>
   <xacro:property name="caster_mass"     value="0.2"/>
-  <xacro:property name="base_mass"       value="8.0"/>
-  <xacro:property name="blade_radius"    value="0.15"/>
-  <xacro:property name="blade_height"    value="0.02"/>
+  <xacro:property name="caster_x_offset" value="0.22"/>
+  <xacro:property name="caster_track"    value="0.36"/>  <!-- centre-to-centre -->
+  <xacro:property name="base_mass"       value="8.76"/>
+  <xacro:property name="blade_radius"    value="0.09"/>
+  <xacro:property name="blade_height"    value="0.01"/>
   <xacro:property name="blade_mass"      value="0.3"/>
   <!-- Derived: base_link is wheel_radius above ground -->
@@ -135,6 +142,6 @@
       <parent link="base_link"/>
       <child  link="${side}_wheel_link"/>
-      <!-- Wheels sit at x=0 (mid-axle), y = ±track/2, z = 0 (ground) -->
-      <origin xyz="0 ${y_reflect * wheel_track/2} 0" rpy="0 0 0"/>
+      <!-- Rear drive wheels: offset behind base_link centre -->
+      <origin xyz="${wheel_x_offset} ${y_reflect * wheel_track/2} 0" rpy="0 0 0"/>
       <axis xyz="0 1 0"/>
       <dynamics damping="0.1" friction="0.1"/>
@@ -152,47 +159,47 @@
   <xacro:drive_wheel side="right" y_reflect="-1"/>
   <!-- ================================================================
-       Front caster
-       ================================================================ -->
-  <link name="front_caster_link">
-    <visual>
-      <origin xyz="0 0 0" rpy="0 0 0"/>
-      <geometry>
-        <sphere radius="${caster_radius}"/>
-      </geometry>
-      <material name="light_grey">
-        <color rgba="0.7 0.7 0.7 1.0"/>
-      </material>
-    </visual>
-    <collision>
-      <origin xyz="0 0 0" rpy="0 0 0"/>
-      <geometry>
-        <sphere radius="${caster_radius}"/>
-      </geometry>
-    </collision>
-    <inertial>
-      <mass value="${caster_mass}"/>
-      <inertia
-        ixx="${(2.0/5.0)*caster_mass*caster_radius*caster_radius}"
-        ixy="0" ixz="0"
-        iyy="${(2.0/5.0)*caster_mass*caster_radius*caster_radius}"
-        iyz="0"
-        izz="${(2.0/5.0)*caster_mass*caster_radius*caster_radius}"/>
-    </inertial>
-  </link>
-  <joint name="front_caster_joint" type="fixed">
-    <parent link="base_link"/>
-    <child  link="front_caster_link"/>
-    <!-- Front of base, at ground level (z = -wheel_radius + caster_radius) -->
-    <origin xyz="${base_length/2 - caster_radius}
-                 0
-                 ${-wheel_radius + caster_radius}"
-            rpy="0 0 0"/>
-  </joint>
-  <gazebo reference="front_caster_link">
-    <mu1>0.0</mu1>
-    <mu2>0.0</mu2>
-    <kp>1e6</kp>
-    <kd>1.0</kd>
-  </gazebo>
+       Front caster wheel macro (two front casters like real robot)
+       ================================================================ -->
+  <xacro:macro name="front_caster" params="side y_reflect">
+    <link name="front_${side}_caster_link">
+      <visual>
+        <origin xyz="0 0 0" rpy="${pi/2} 0 0"/>
+        <geometry>
+          <cylinder radius="${caster_radius}" length="${caster_width}"/>
+        </geometry>
+        <material name="dark_grey"/>
+      </visual>
+      <collision>
+        <origin xyz="0 0 0" rpy="${pi/2} 0 0"/>
+        <geometry>
+          <cylinder radius="${caster_radius}" length="${caster_width}"/>
+        </geometry>
+      </collision>
+      <inertial>
+        <mass value="${caster_mass}"/>
+        <inertia
+          ixx="${(2.0/5.0)*caster_mass*caster_radius*caster_radius}"
+          ixy="0" ixz="0"
+          iyy="${(2.0/5.0)*caster_mass*caster_radius*caster_radius}"
+          iyz="0"
+          izz="${(2.0/5.0)*caster_mass*caster_radius*caster_radius}"/>
+      </inertial>
+    </link>
+    <joint name="front_${side}_caster_joint" type="continuous">
+      <parent link="base_link"/>
+      <child  link="front_${side}_caster_link"/>
+      <!-- Front casters: forward of centre, z at ground level -->
+      <origin xyz="${caster_x_offset} ${y_reflect * caster_track/2} ${-wheel_radius + caster_radius}" rpy="0 0 0"/>
+      <axis xyz="0 1 0"/>
+    </joint>
+    <gazebo reference="front_${side}_caster_link">
+      <mu1>0.0</mu1>
+      <mu2>0.0</mu2>
+      <kp>1e6</kp>
+      <kd>1.0</kd>
+    </gazebo>
+  </xacro:macro>
+  <xacro:front_caster side="left"  y_reflect="1"/>
+  <xacro:front_caster side="right" y_reflect="-1"/>
   <!-- ================================================================
        Blade disc  (centred under base, just below chassis)
@@ -200,5 +207,5 @@
   <link name="blade_link">
     <visual>
-      <origin xyz="0 0 0" rpy="0 0 0"/>
+      <origin xyz="0 0 ${blade_height/2}" rpy="0 0 0"/>
       <geometry>
         <cylinder radius="${blade_radius}" length="${blade_height}"/>
@@ -218,9 +225,10 @@
                             h="${blade_height}"/>
   </link>
-  <joint name="blade_joint" type="fixed">
+  <joint name="blade_joint" type="continuous">
     <parent link="base_link"/>
     <child  link="blade_link"/>
-    <!-- Hang blade flush below the chassis floor -->
-    <origin xyz="0 0 ${-(blade_height/2)}" rpy="0 0 0"/>
+    <!-- Blade disc centred under base, matching real robot -->
+    <origin xyz="0 0 ${-wheel_radius + 0.05}" rpy="0 0 0"/>
+    <axis xyz="0 0 1"/>
   </joint>
   <!-- ================================================================
@@ -316,5 +324,6 @@
     <parent link="base_link"/>
     <child  link="lidar_link"/>
-    <origin xyz="0.20 0 0.25" rpy="0 0 0"/>
+    <!-- Mounted on top front of chassis -->
+    <origin xyz="0.20 0 ${base_height + 0.03}" rpy="0 0 0"/>
   </joint>
   <!-- ================================================================

Commit message: feat: configurable lidar position and orientation via mowgli_robot.yaml
The lidar_joint transform in the URDF was hardcoded. Now lidar_x,
lidar_y, lidar_z, lidar_yaw are read from mowgli_robot.yaml and
passed as xacro arguments, so users can adjust the lidar mounting
position and orientation without rebuilding the image.

File: src/mowgli_bringup/urdf/mowgli.urdf.xacro (robot description, xacro)
@@ -17,4 +17,11 @@
 -->
 <robot name="mowgli" xmlns:xacro="http://www.ros.org/wiki/xacro">
+  <!-- ================================================================
+       Configurable arguments (can be overridden via xacro command-line)
+       ================================================================ -->
+  <xacro:arg name="lidar_x"   default="0.20"/>
+  <xacro:arg name="lidar_y"   default="0.0"/>
+  <xacro:arg name="lidar_z"   default="0.22"/>
+  <xacro:arg name="lidar_yaw" default="0.0"/>
   <!-- ================================================================
        Properties
@@ -324,6 +331,6 @@
     <parent link="base_link"/>
     <child  link="lidar_link"/>
-    <!-- Mounted on top front of chassis -->
-    <origin xyz="0.20 0 ${base_height + 0.03}" rpy="0 0 0"/>
+    <!-- Mounted on top front of chassis — position configurable via xacro args -->
+    <origin xyz="$(arg lidar_x) $(arg lidar_y) $(arg lidar_z)" rpy="0 0 $(arg lidar_yaw)"/>
   </joint>
   <!-- ================================================================
